Commit message: correct base_link offset to footprint

File: urdf/youbot_base/base.urdf.xacro (robot description, xacro)
@@ -38,5 +38,5 @@
     		</link>
     		<joint name="${name}_footprint_joint" type="fixed">
-      			<origin xyz="0 0 0" rpy="0 0 0" />
+      			<origin xyz="0 0 ${-wheel_offset_z + wheel_radius}" rpy="0 0 0" />
       			<child link="${name}_link" />
       			<parent link="${name}_footprint"/>
