Commit message: include profile frame and x4 Lidar to description

File: robots/youbot.urdf.xacro (robot description, xacro)
@@ -12,6 +12,8 @@
   <!-- youbot gripper -->
   <xacro:include filename="$(find youbot_description)/urdf/youbot_gripper/gripper.urdf.xacro" />
-  <!-- joint state publisher -->
-  <xacro:include filename="$(find youbot_description)/robots/youbot_gazebo.xacro" />
+  <!-- youbot profile frame -->
+  <xacro:include filename="$(find youbot_description)/urdf/youbot_profile_frame/profiles.urdf.xacro" />
+  <!-- youbot X4 LiDAR -->
+  <xacro:include filename="$(find youbot_description)/urdf/sensors/X4.urdf.xacro" />
   <!-- Now we can start using the macros included above to define the actual youbot -->
   <xacro:youbot_base name="base" namespace=""/>
@@ -21,19 +23,18 @@
   <xacro:youbot_arm name="arm" parent="base_link" namespace="">
     <origin xyz="0.135 0.0 0.051" rpy="0 0 0" />
-    <!--<origin xyz="0.258 0 0.066" rpy="0 0 0.576" />-->
-    <!--Default inertia to see if jittering stops-->
-    <!--<inertia ixx="0.1" ixy="0" ixz="0" iyy="0.1" iyz="0" izz="0.1" />-->
   </xacro:youbot_arm>
   <xacro:youbot_gripper name="gripper" parent="arm_link_5" namespace="">
     <origin xyz="0 0 0" rpy="0 0 0" />
-    <!--Default inertia to see if jittering stops-->
-    <!--<inertia ixx="0.1" ixy="0" ixz="0" iyy="0.1" iyz="0" izz="0.1" />-->
   </xacro:youbot_gripper>
+  <xacro:youbot_profile_frame name="profiles" parent="base_link">
+    <origin xyz="0.0 0 0.0307" rpy="0 0 0" /> <!-- profiles origin frme is on the base upper surface of the base plate-->
+  </xacro:youbot_profile_frame>
+  <xacro:x4 name="x4" parent="base_link">
+    <origin xyz="-0.369 0 0.0447" rpy="0 0 0" /> <!-- profiles origin frme is on the base upper surface of the base plate-->
+  </xacro:x4>
   <!-- Kamera -->
   <!--xacro:include filename="$(find youbot_description)/urdf/sensors/asus_xtion_camera.urdf.xacro" />
   <xacro:asus_xtion_camera name="camera" parent="arm_link_5" tilt="0.0">
     <origin xyz="-0.02 0 -0.04" rpy="0 -1.60 0" />
-    <inertia ixx="0.1" ixy="0" ixz="0" iyy="0.1" iyz="0" izz="0.1" />
   </xacro:asus_xtion_camera-->
-  <xacro:joint_state_publisher namespace="gazebo"/>
 </robot>

Commit message: insert camera and correct position

File: robots/youbot.urdf.xacro (robot description, xacro)
@@ -34,7 +34,7 @@
   </xacro:x4>
   <!-- Kamera -->
-  <!--xacro:include filename="$(find youbot_description)/urdf/sensors/asus_xtion_camera.urdf.xacro" />
+  <xacro:include filename="$(find youbot_description)/urdf/sensors/asus_xtion_camera.urdf.xacro" />
   <xacro:asus_xtion_camera name="camera" parent="arm_link_5" tilt="0.0">
-    <origin xyz="-0.02 0 -0.04" rpy="0 -1.60 0" />
-  </xacro:asus_xtion_camera-->
+    <origin xyz="-0.04 0 -0.0086" rpy="0 -1.60 0" />
+  </xacro:asus_xtion_camera>
 </robot>

File: urdf/youbot_arm/arm.urdf.xacro (robot description, xacro)
@@ -168,5 +168,5 @@
 		<!-- joint between arm_4_link and arm_5_link -->
 		<joint name="${name}_joint_5" type="revolute">
-			<origin xyz="-0.002 0 0.130" rpy="0 0 ${167.5 * M_PI / 180}" />
+			<origin xyz="-0.002 0 0.147" rpy="0 0 ${167.5 * M_PI / 180}" />
 			<parent link="${name}_link_4"/>
 			<child link="${name}_link_5"/>

Commit message: Change z-offset of x4 sensor

File: robots/youbot.urdf.xacro (robot description, xacro)
@@ -28,8 +28,8 @@
   </xacro:youbot_gripper>
   <xacro:youbot_profile_frame name="profiles" parent="base_link">
-    <origin xyz="0.0 0 0.0307" rpy="0 0 0" /> <!-- profiles origin frme is on the base upper surface of the base plate-->
+    <origin xyz="0.0 0 0.044" rpy="0 0 0" /> <!-- profiles origin frme is on the base upper surface of the base plate-->
   </xacro:youbot_profile_frame>
   <xacro:x4 name="x4" parent="base_link">
-    <origin xyz="-0.369 0 0.0447" rpy="0 0 0" /> <!-- profiles origin frme is on the base upper surface of the base plate-->
+    <origin xyz="-0.369 0 0.058" rpy="0 0 0" /> <!-- profiles origin frme is on the base upper surface of the base plate-->
   </xacro:x4>
   <!-- Kamera -->

Commit message: Add aruco marker to description

File: robots/youbot.urdf.xacro (robot description, xacro)
@@ -16,4 +16,6 @@
   <!-- youbot X4 LiDAR -->
   <xacro:include filename="$(find youbot_description)/urdf/sensors/X4.urdf.xacro" />
+  <!-- youbot aruco marker on X4 LiDAR -->
+  <xacro:include filename="$(find youbot_description)/urdf/aruco_marker/aruco_marker_0.urdf.xacro" />
   <!-- Now we can start using the macros included above to define the actual youbot -->
   <xacro:youbot_base name="base" namespace=""/>
@@ -30,4 +32,5 @@
     <origin xyz="0.0 0 0.044" rpy="0 0 0" /> <!-- profiles origin frme is on the base upper surface of the base plate-->
   </xacro:youbot_profile_frame>
+  <!-- LiDAR -->
   <xacro:x4 name="x4" parent="base_link">
     <origin xyz="-0.369 0 0.058" rpy="0 0 0" /> <!-- profiles origin frme is on the base upper surface of the base plate-->
@@ -36,5 +39,9 @@
   <xacro:include filename="$(find youbot_description)/urdf/sensors/asus_xtion_camera.urdf.xacro" />
   <xacro:asus_xtion_camera name="camera" parent="arm_link_5" tilt="0.0">
-    <origin xyz="-0.04 0 -0.0086" rpy="0 -1.60 0" />
+    <origin xyz="-0.011 -0.02 -0.0286" rpy="0 -1.60 0" />
   </xacro:asus_xtion_camera>
+  <!-- aruco marker on LiDAR -->
+  <xacro:aruco_marker_0 name="aruco_marker_0" parent="x4_plate_link">
+    <origin xyz="0 0 0.005" rpy="0 0 0" /> <!-- profiles origin frme is on the base upper surface of the base plate-->
+  </xacro:aruco_marker_0>
 </robot>

Commit message: Adapt camera position

File: robots/youbot.urdf.xacro (robot description, xacro)
@@ -39,5 +39,5 @@
   <xacro:include filename="$(find youbot_description)/urdf/sensors/asus_xtion_camera.urdf.xacro" />
   <xacro:asus_xtion_camera name="camera" parent="arm_link_5" tilt="0.0">
-    <origin xyz="-0.011 -0.02 -0.0286" rpy="0 -1.60 0" />
+    <origin xyz="-0.03 -0.002 -0.023" rpy="0 -1.60 0" />
   </xacro:asus_xtion_camera>
   <!-- aruco marker on LiDAR -->
